File: hardware/panelized/fk-sonar-v0.07-03x03.kicad_pcb (KiCad board)
At the start: 4 copper layers, 34.5 x 70.5 mm, 73 parts, among them J1 CONN_01x03, J10 CONN_01x05, J11 CONN_01x04, J12 CONN_01x04, J13 CONN_01x04, J2 CONN_02x05_SWD, J3 MICRO-USB, J4 MICRO-USB, J5 CONN_01x02, J6 CONN_01x04, J7 CONN_01x02, J8 CONN_01x03_SERIAL, J9 CONN_01x05, M1 MOUNT_HOLE, M2 FIDUCIAL, M3 MOUNT_HOLE, M4 MOUNT_HOLE, M5 FIDUCIAL, M6 MOUNT_HOLE, Q1 2N7002LT1G, SW1 SPNO, U1 ATSAMD21G18A-AU, U2 MCP1700T-3302E/MB, U3 TPS2052B, U4 S25FL116K0XMFI041, U7 SK6812, Y1 FC-135

Commit message: Changed board outline slightly to be on a 0.5 mm grid (for panelization)
Parts:
- added P2: ATLAS_EC_PROBE, conservify:Dummy_Empty, F.Cu at (442.3, 113.8)
- added P3: ATLAS_RTD_PROBE, conservify:Dummy_Empty, F.Cu at (442.3, 113.8)
- added P4: ATLAS_PH_PROBE, conservify:Dummy_Empty, F.Cu at (442.3, 113.8)
- added P5: ATLAS_DO_PROBE, conservify:Dummy_Empty, F.Cu at (442.3, 113.8)
- added P6: ATLAS_ORP_PROBE, conservify:Dummy_Empty, F.Cu at (442.3, 113.8)
- added REF**: MouseBite, Utah-Blink-FP:MouseBite, B.Cu at (120.7, 79.2)
Other:
- board size 34.5 x 70.5 mm -> 98 x 73.5 mm
- board text added: "CORE"
- board text removed: "IBB"
Changed lines of the file:
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@@
   (general
     (thickness 1.6)
-    (drawings 25)
+    (drawings 28)
     (tracks 671)
     (zones 0)
-    (modules 73)
+    (modules 79)
     (nets 70)
   )
@@
     (46 B.CrtYd user)
     (47 F.CrtYd user)
-    (48 B.Fab user hide)
-    (49 F.Fab user hide)
+    (48 B.Fab user)
+    (49 F.Fab user)
   )
   (setup
@@
     (user_trace_width 0.762)
     (user_trace_width 1.27)
+    (user_trace_width 0.3048)
+    (user_trace_width 0.6096)
+    (user_trace_width 0.2032)
+    (user_trace_width 0.254)
+    (user_trace_width 0.381)
+    (user_trace_width 0.508)
+    (user_trace_width 0.762)
+    (user_trace_width 1.27)
+    (user_trace_width 0.203)
+    (user_trace_width 0.381)
+    (user_trace_width 0.587)
+    (user_trace_width 0.762)
+    (user_trace_width 0.2032)
+    (user_trace_width 0.254)
+    (user_trace_width 0.381)
+    (user_trace_width 0.508)
+    (user_trace_width 0.762)
+    (user_trace_width 1.27)
     (trace_clearance 0.1524)
     (zone_clearance 0.2032)
@@
     (pad_drill 0)
     (pad_to_mask_clearance 0)
+    (solder_mask_min_width 0.25)
     (pad_to_paste_clearance_ratio -0.05)
     (aux_axis_origin 127 127)
-    (grid_origin 122.17 62.23)
+    (grid_origin 184.4514 104.9894)
     (visible_elements 7FFFDF7F)
     (pcbplotparams
@@
     (add_net VUSB)
   )
+  (module Utah-Blink-FP:MouseBite (layer B.Cu)
+    (at 120.6714 79.2294 90)
+    (fp_text reference REF** (at 0 -0.5 90) (layer B.SilkS) hide
+      (effects (font (size 1 1) (thickness 0.15)) (justify mirror))
+    )
+    (fp_text value MouseBite (at 0 2.7 90) (layer B.Fab) hide
+      (effects (font (size 1 1) (thickness 0.15)) (justify mirror))
+    )
+    (fp_line (start -1.5 -1.5) (end -1.5 1.5) (layer Dwgs.User) (width 0.15))
+    (fp_line (start 1.5 1.5) (end 1.5 -1.5) (layer Dwgs.User) (width 0.15))
+    (pad "" np_thru_hole circle (at -1.2 -1.5 90) (size 0.5 0.5) (drill 0.5) (layers *.Cu *.Mask))
+    (pad "" np_thru_hole circle (at 0 -1.5 90) (size 0.5 0.5) (drill 0.5) (layers *.Cu *.Mask))
+    (pad "" np_thru_hole circle (at 1.2 -1.5 90) (size 0.5 0.5) (drill 0.5) (layers *.Cu *.Mask))
+    (pad "" np_thru_hole circle (at 1.2 1.5 90) (size 0.5 0.5) (drill 0.5) (layers *.Cu *.Mask))
+    (pad "" np_thru_hole circle (at 0 1.5 90) (size 0.5 0.5) (drill 0.5) (layers *.Cu *.Mask))
+    (pad "" np_thru_hole circle (at -1.2 1.5 90) (size 0.5 0.5) (drill 0.5) (layers *.Cu *.Mask))
+  )
   (module conservify:SOIC-8-N (layer F.Cu)
     (at 144.7038 114.1476 270)
@@
       (net 5 /RST))
   )
-  (module conservify:conservify_text_negative_5000 locked (layer F.Cu)
+  (module conservify:conservify_text_negative_5000 (layer F.Cu)
     (at 147.8915 70.739)
     (fp_text reference G*** (at 0 0) (layer F.SilkS) hide
@@
       (xy -5.181097 -1.438992)) (layer F.SilkS) (width 0.01))
   )
-  (module conservify:osh_negative_3000 locked (layer F.Cu)
+  (module conservify:osh_negative_3000 (layer F.Cu)
     (at 151.13 64.516)
     (fp_text reference G*** (at 0 0) (layer F.SilkS) hide
@@
     )
   )
-  (module conservify:LOGO_FK_NEGATIVE_2500 locked (layer F.Cu)
+  (module conservify:LOGO_FK_NEGATIVE_2500 (layer F.Cu)
     (at 151.1935 73.025)
     (fp_text reference G*** (at 0 0) (layer F.SilkS) hide
@@
       (xy -1.681029 -0.402171) (xy -1.625433 -0.40388) (xy -1.568308 -0.402711)) (layer F.SilkS) (width 0.01))
   )
-  (gr_arc (start 123.17 63.23) (end 123.17 62.23) (angle -90) (layer Edge.Cuts) (width 0.15))
-  (gr_line (start 122.17 131.73) (end 122.17 63.23) (layer Edge.Cuts) (width 0.15))
+  (module conservify:Dummy_Empty (layer F.Cu)
+    (at 442.2918 113.808601)
+    (descr "Only empty Dummy to give satsfaction to DRC")
+    (tags "Only empty Dummy to give satsfaction to DRC")
+    (fp_text reference P2 (at 2.5654 -1.007201) (layer F.SilkS) hide
+      (effects (font (size 1 1) (thickness 0.15)))
+    )
+    (fp_text value ATLAS_EC_PROBE (at 0 0) (layer F.Fab) hide
+      (effects (font (size 1 1) (thickness 0.15)))
+    )
+  )
+  (module conservify:Dummy_Empty (layer F.Cu)
+    (at 442.2918 113.808601)
+    (descr "Only empty Dummy to give satsfaction to DRC")
+    (tags "Only empty Dummy to give satsfaction to DRC")
+    (fp_text reference P3 (at 3.1242 -1.185001) (layer F.SilkS) hide
+      (effects (font (size 1 1) (thickness 0.15)))
+    )
+    (fp_text value ATLAS_RTD_PROBE (at 0 0) (layer F.Fab) hide
+      (effects (font (size 1 1) (thickness 0.15)))
+    )
+  )
+  (module conservify:Dummy_Empty (layer F.Cu)
+    (at 442.2918 113.808601)
+    (descr "Only empty Dummy to give satsfaction to DRC")
+    (tags "Only empty Dummy to give satsfaction to DRC")
+    (fp_text reference P4 (at 2.413 -3.648801) (layer F.SilkS) hide
+      (effects (font (size 1 1) (thickness 0.15)))
+    )
+    (fp_text value ATLAS_PH_PROBE (at 0 0) (layer F.Fab) hide
+      (effects (font (size 1 1) (thickness 0.15)))
+    )
+  )
+  (module conservify:Dummy_Empty (layer F.Cu)
+    (at 442.2918 113.808601)
+    (descr "Only empty Dummy to give satsfaction to DRC")
+    (tags "Only empty Dummy to give satsfaction to DRC")
+    (fp_text reference P5 (at 2.54 -5.096601) (layer F.SilkS) hide
+      (effects (font (size 1 1) (thickness 0.15)))
+    )
+    (fp_text value ATLAS_DO_PROBE (at 0 0) (layer F.Fab) hide
+      (effects (font (size 1 1) (thickness 0.15)))
+    )
+  )
+  (module conservify:Dummy_Empty (layer F.Cu)
+    (at 442.2918 113.808601)
+    (descr "Only empty Dummy to give satsfaction to DRC")
+    (tags "Only empty Dummy to give satsfaction to DRC")
+    (fp_text reference P6 (at 3.429 0.643799) (layer F.SilkS) hide
+      (effects (font (size 1 1) (thickness 0.15)))
+    )
+    (fp_text value ATLAS_ORP_PROBE (at 0 0) (layer F.Fab) hide
+      (effects (font (size 1 1) (thickness 0.15)))
+    )
+  )
+  (gr_line (start 122.17 131.73) (end 122.17 80.73) (layer Edge.Cuts) (width 0.15))
   (gr_arc (start 123.17 131.73) (end 122.17 131.73) (angle -90) (layer Edge.Cuts) (width 0.15))
   (gr_line (start 155.67 132.73) (end 123.17 132.73) (layer Edge.Cuts) (width 0.15))
   (gr_arc (start 155.67 131.73) (end 155.67 132.73) (angle -90) (layer Edge.Cuts) (width 0.15))
-  (gr_line (start 156.67 63.73) (end 156.67 131.73) (layer Edge.Cuts) (width 0.15))
+  (gr_line (start 156.67 63.23) (end 156.67 131.73) (layer Edge.Cuts) (width 0.15))
   (gr_arc (start 155.67 63.23) (end 156.67 63.23) (angle -90) (layer Edge.Cuts) (width 0.15))
   (gr_line (start 123.17 62.23) (end 155.67 62.23) (layer Edge.Cuts) (width 0.15))
+  (gr_line (start 122.17 63.23) (end 122.17 77.73) (layer Edge.Cuts) (width 0.15))
+  (gr_line (start 119.17 59.23) (end 217.17 59.23) (layer Edge.Cuts) (width 0.15))
   (gr_text PWR (at 149.7965 92.9005) (layer F.SilkS)
     (effects (font (size 0.762 0.762) (thickness 0.1524)))
@@
     (effects (font (size 0.762 0.762) (thickness 0.1524)))
   )
-  (gr_text IBB (at 124.841 79.883) (layer F.SilkS)
+  (gr_text CORE (at 124.841 79.883) (layer F.SilkS)
     (effects (font (size 1 1) (thickness 0.2)))
   )
@@
     (effects (font (size 0.762 0.762) (thickness 0.1524)))
   )
+  (gr_arc (start 123.19 63.246) (end 122.174 63.246) (angle 90) (layer Edge.Cuts) (width 0.15))
+  (gr_arc (start 155.702 63.246) (end 155.67 62.23) (angle 0.0001126752005) (layer Edge.Cuts) (width 0.15))
   (via (at 136.144 72.517) (size 0.5) (drill 0.3) (layers F.Cu B.Cu) (net 1))
   (via (at 135.128 72.517) (size 0.5) (drill 0.3) (layers F.Cu B.Cu) (net 1))
